File: pcb/RP2040_CO2_sensor/RP2040_CO2_sensor.kicad_pcb (KiCad board)
At the start: 2 copper layers, 35.6 x 30.5 mm, 13 parts, among them J1 Conn_01x04_Female, J2 Conn_01x04_Female, J3 Conn_01x08_Female, J4 Conn_01x08_Female, J5 Conn_01x04_Female, J6 Conn_01x05_Female, J7 Conn_01x03_Female, J8 Conn_01x04_Female

Commit message: :sparkles: add PCB
Parts:
- removed the G*** at (109.9, 106.0)
- added G***: LOGO, logo_silk:logo_toms_85x40_silk, F.Cu at (95.2, 117.5)
- added G***: LOGO, lib:logo_co2mo_mask, F.Cu at (109.9, 106.0)
Routing:
- net /GPIO7: track 0.00 -> 39.9 mm
- net /GPIO6: track 0.00 -> 36.9 mm
- net +3V3: track 0.00 -> 32.0 mm
- net /GPIO3: track 0.00 -> 28.7 mm
- net /GPIO2: track 0.00 -> 26.2 mm
- net +5V: track 0.00 -> 25.6 mm
- net /A3: track 0.00 -> 15.9 mm
- net /RX: track 0.00 -> 13.9 mm
- net /A0: track 0.00 -> 13.4 mm
- net /TX: track 0.00 -> 12.7 mm
- net GND: track 0.00 -> 12.2 mm, vias 0 -> 11
- net /SDA: track 0.00 -> 8.67 mm
- net /SCL: track 0.00 -> 8.67 mm
- net /A2: track 0.00 -> 7.18 mm
- net /A1: track 0.00 -> 5.08 mm
- added copper zone on B.Cu, net GND
- added copper zone on F.Cu, net GND
Other:
- board text added: "Tiny2040"
